File: 1_hardware_PCB/MainBoard_Damashi/MainBoard_Damashi.kicad_pcb (KiCad board)
At the start: 2 copper layers, 70 x 55 mm, 27 parts, among them J10 Aux 1, J11 Aux 2, J12 JST-CNY70, J3 STEP_DOWN, J5 Left, J6 JST-CNY70, J7 Mid, J8 JST-CNY70, J9 Right, P1 Mounting_Hole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

Commit message: Diseñe el PCB
Parts:
- removed D1: LED, EESTN5:led_5mm_clear
- removed G***: LOGO, Falconlogos:Mini logo 2
- removed J11: Aux 2, Connector:FanPinHeader_1x03_P2.54mm_Vertical
- removed J12, J6: JST-CNY70, Connector:FanPinHeader_1x03_P2.54mm_Vertical
- removed J9: Right, Connector:FanPinHeader_1x03_P2.54mm_Vertical
- removed R1: 4K7, EESTN5:RES0.3
- removed SW1, SW2: START, Connector_PinHeader_2.54mm:PinHeader_1x02_P2.54mm_Horizontal
- removed U4: ESP32_DevKit_V1_CH9102X, EESTN5:ESP32_DevKit_V1_CH9102X
- added J1: STEP_DOWN, Connector_PinHeader_2.54mm:PinHeader_1x02_P2.54mm_Horizontal, F.Cu at (131.0, 79.7)
- added J2: Buttons, Connector_PinHeader_2.54mm:PinHeader_1x02_P2.54mm_Horizontal, F.Cu at (102.1, 110.3)
- added J4: Aux 1, Connector:FanPinHeader_1x03_P2.54mm_Vertical, F.Cu at (117.9, 71.2)
- added U1: ESP32_DevKit_V1_CH9102X, EESTN5:ESP32_DevKit_V1_CH9102X, F.Cu at (103.3, 94.2)
- D2: footprint EESTN5:led_5mm_clear -> Connector_PinHeader_2.54mm:PinHeader_1x02_P2.54mm_Horizontal
- J10: value Aux 1 -> Qre1113_Conn; footprint Connector:FanPinHeader_1x03_P2.54mm_Vertical -> Connector_PinHeader_2.54mm:PinHeader_1x05_P2.54mm_Horizontal
- J3: value STEP_DOWN -> Left; footprint EESTN5:BORNERA3_AZUL -> Connector:FanPinHeader_1x03_P2.54mm_Vertical
- J5: value Left -> Mid
- J7: value Mid -> Aux 2
- J8: value JST-CNY70 -> Right
- Q1: moved to B.Cu
- R2: value 4K7 -> 220; footprint EESTN5:RES0.3 -> EESTN5:R_1206; moved to B.Cu
- R3: value 220 -> 10K; moved to B.Cu
- R4: value 220 -> 4K7; moved to B.Cu
- R5: value 10K -> 4K7; moved to B.Cu
- moved R5 163.3 mm to (91.5, 103.3), turned to 180 degrees
- moved R4 163.2 mm to (91.5, 100.7), turned to 180 degrees
- moved P1 153.4 mm to (79.6, 74.7)
- moved R3 148.5 mm to (105.9, 103.2)
- moved D2 135.5 mm to (117.1, 91.5)
- moved BZ1 131.7 mm to (110.9, 99.0), turned to 90 degrees
- moved P4 130.9 mm to (87.1, 113.5)
- moved P3 121.0 mm to (110.8, 113.8)
- moved J10 116.0 mm to (86.6, 96.5), turned to 180 degrees
- moved P2 107.7 mm to (125.5, 83.5)
- moved J8 94.1 mm to (96.3, 71.2), turned to -90 degrees
- moved Q1 92.3 mm to (108.3, 98.8)
- moved P5 91.1 mm to (125.9, 113.5), turned to 180 degrees
- moved J3 91.0 mm to (110.8, 71.2), turned to -90 degrees
- moved R2 90.6 mm to (102.0, 102.7), turned to -90 degrees
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Connections:
- J10 pad 1: +5V -> /TATAMI_B
- J10 pad 2: GND -> /TATAMI_L
- J10 pad 3: /AUX_DISTANCE_1 -> /TATAMI_R
- J3 pad 1: /Vstep -> +5V
- J3 pad 3: +5V -> /L_DISTANCE
- J5 pad 3: /L_DISTANCE -> /M_DISTANCE
- J7 pad 3: /M_DISTANCE -> /AUX_DISTANCE_2
- J8 pad 3: /TATAMI_R -> /R_DISTANCE
- R2 pad 1: +3V3 -> /LED_1
- R2 pad 2: /PUSH_2 -> Net-(D2-A)
- R3 pad 1: /LED_2 -> Net-(Q1-G)
- R3 pad 2: Net-(D1-A) -> /BUZZER
- R4 pad 1: /LED_1 -> +3V3
- R4 pad 2: Net-(D2-A) -> /PUSH_1
- R5 pad 1: Net-(Q1-G) -> +3V3
- R5 pad 2: /BUZZER -> /PUSH_2
Routing:
- net GND: track 125.1 -> 0.00 mm
- net (no net): track 27.2 -> 0.00 mm
- net /TATAMI_B: track 0.00 -> 23.6 mm
- net Net-(D2-A): track 0.00 -> 23.5 mm
- net /AUX_DISTANCE_2: track 0.00 -> 16.8 mm
- net /PUSH_1: track 0.00 -> 16.3 mm
- net +5V: track 185.9 -> 201.7 mm
- net /M2B: track 20.9 -> 5.80 mm
- net /PUSH_2: track 0.00 -> 12.6 mm
- net /AUX_DISTANCE_1: track 0.00 -> 11.1 mm
- net /M1B: track 11.5 -> 22.4 mm
- net +3V3: track 21.4 -> 11.0 mm
- net /Vstep: track 8.90 -> 0.00 mm
- net /TATAMI_L: track 12.7 -> 19.8 mm
- net Net-(BZ1-+): track 0.00 -> 5.31 mm
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Other:
- board size 70 x 55 mm -> 60 x 50 mm
