File: 1_hardware_PCB/MainBoard_Damashi/MainBoard_Damashi.kicad_sch (KiCad schematic)
At the start: 26 parts, among them J10 Aux 1, J11 Aux 2, J12 JST-CNY70, J3 STEP_DOWN, J5 Left, J6 JST-CNY70, J7 Mid, J8 JST-CNY70, J9 Right, P1 Mounting_Hole, P2 Mounting_Hole, P3 Mounting_Hole, P4 MOTOR_DER, P5 MOTOR_IZQ, Q1 2N7002, SW1 START, SW2 START, U4 ESP32_DevKit_V1_CH9102X

Commit message: Diseñe el PCB
Parts:
- removed D1: LED, EESTN5:led_5mm_clear, symbol Device:LED
- removed J12, J6, J8: JST-CNY70, Connector:FanPinHeader_1x03_P2.54mm_Vertical, symbol 2019---Sumo---NANO---BTS7960-rescue:Conn_01X03-EESTN5
- removed J3: STEP_DOWN, EESTN5:BORNERA3_AZUL, symbol 2019---Sumo---NANO---BTS7960-rescue:TB_1X3-EESTN5
- removed R3: 220, EESTN5:R_1206, symbol Device:R
- removed SW1, SW2: START, Connector_PinHeader_2.54mm:PinHeader_1x02_P2.54mm_Horizontal, symbol 2019---Sumo---NANO---BTS7960-rescue:SW_Push-EESTN5
- added J1: STEP_DOWN, Connector_PinHeader_2.54mm:PinHeader_1x02_P2.54mm_Horizontal, symbol Connector:Conn_01x02_Pin
- added J10: Qre1113_Conn, Connector_PinHeader_2.54mm:PinHeader_1x05_P2.54mm_Horizontal, symbol Connector:Conn_01x05_Pin
- added J2: Buttons, Connector_PinHeader_2.54mm:PinHeader_1x02_P2.54mm_Horizontal, symbol Connector:Conn_01x02_Pin
- D2: footprint EESTN5:led_5mm_clear -> Connector_PinHeader_2.54mm:PinHeader_1x02_P2.54mm_Horizontal
- R4: renamed from R1; footprint EESTN5:RES0.3 -> EESTN5:R_1206
- R5: renamed from R2; footprint EESTN5:RES0.3 -> EESTN5:R_1206
- renumbered J5 to J3, J10 to J4, J7 to J5, J11 to J7, J9 to J8, R4 to R2, R5 to R3, U4 to U1
Connections:
- net +5V: now also J1.2 (Pin_2), J10.5 (Pin_5)
- net AUX_DISTANCE_2: now also U1.4 (IO34); no longer U1.9 (IO26)
- net GND: now also J1.1 (Pin_1), J10.4 (Pin_4)
- net PUSH_1: now also U1.22 (TX2), J2.1 (Pin_1); no longer U1.21 (RX2)
- net PUSH_2: now also U1.21 (RX2), J2.2 (Pin_2); no longer U1.22 (TX2)
- net TATAMI_B: now also U1.9 (IO26), J10.1 (Pin_1); no longer U1.13 (IO13)
- net TATAMI_L: now also U1.10 (IO27), J10.2 (Pin_2); no longer U1.4 (IO34)
- net TATAMI_R: now also U1.13 (IO13), J10.3 (Pin_3); no longer U1.10 (IO27)
- net LED_2: no longer names the net of U1.20 (IO4)
